File: pcb/ES-Seed3-DevKit-Desktop-Rev1/Seed3-DevKit-Desktop_1.kicad_sch (KiCad schematic)
At the start: 71 parts, among them J7 USB4110GFA, U1 TL072, U12 CD4051B, U13 TL072, U14 USBLC6-2SC6, U15 TL072, U2 MCP6004

Commit message: schematic is like 85% done.. just needs audio circuits, and opamp choice(s).
Parts:
- removed C16, C18: 1NF, Capacitor_SMD:C_0603_1608Metric, symbol Device:C
- removed J_CV_IN_3, J_CV_IN_4: ~, Electrosmith-Interface:S_JACK, symbol Electrosmith-Interface:EURO_JACK
- removed R35, R36, R39, R45: 200K, Resistor_SMD:R_0603_1608Metric, symbol Seed3-Pedal-DevKit-Converted-eagle-import:Electrosmith-Passives_R-US_R0603
- removed R41, R46: 100K, Resistor_SMD:R_0603_1608Metric, symbol Seed3-Pedal-DevKit-Converted-eagle-import:Electrosmith-Passives_R-US_R0603
- removed R42, R47: 33K, Resistor_SMD:R_0603_1608Metric, symbol Seed3-Pedal-DevKit-Converted-eagle-import:Electrosmith-Passives_R-US_R0603
- removed U1, U13, U15: TL072, Package_SO:SO-8_3.9x4.9mm_P1.27mm, symbol Amplifier_Operational:TL072
- removed U2: MCP6004, Package_SO:SO-14_3.9x8.65mm_P1.27mm, symbol Amplifier_Operational:MCP6004
- added C10, C7, C8: 100NF, Capacitor_SMD:C_0603_1608Metric, symbol Device:C
- added C11: 2.2NF, Capacitor_SMD:C_0603_1608Metric, symbol Device:C
- added C12: 100PF, Capacitor_SMD:C_0603_1608Metric, symbol Device:C
- added C2, C46, C49, C9: 100UF, Capacitor_SMD:CP_Elec_6.3x7.7, symbol Device:C_Polarized_US
- added L1: 1mH, symbol Device:L
- added R32, R5: 10K, Resistor_SMD:R_0603_1608Metric, symbol Seed3-Pedal-DevKit-Converted-eagle-import:Electrosmith-Passives_R-US_R0603
- added R7: 33K, Resistor_SMD:R_0603_1608Metric, symbol Seed3-Pedal-DevKit-Converted-eagle-import:Electrosmith-Passives_R-US_R0603
- added R76, R8: 100K, Resistor_SMD:R_0603_1608Metric, symbol Seed3-Pedal-DevKit-Converted-eagle-import:Electrosmith-Passives_R-US_R0603
- added R77: 10K, Resistor_SMD:R_0603_1608Metric, symbol Device:R_US
- added R81, R83: 47K, Resistor_SMD:R_0603_1608Metric, symbol Device:R_US
- added R82: 150R, Resistor_SMD:R_0603_1608Metric, symbol Device:R_US
- added R84: 100R, Resistor_SMD:R_0603_1608Metric, symbol Device:R_US
- added R9: 3R3, Resistor_SMD:R_1206_3216Metric, symbol Seed3-Pedal-DevKit-Converted-eagle-import:Electrosmith-Passives_R-US_R0603
- added U1, U2, U6: MCP6002-xSN, symbol Amplifier_Operational:MCP6002-xSN
- added U4, U5: 4021, symbol 4xxx:4021
Connections:
- net -12V is gone; now on net GND: C20.2, C3.1, C5.1
- net CV_4_ADC is gone; now on net TOG_1: A1.26 (ADC_4)
- net GPIO_GATEIN_2 is gone; now on net CV_2_ADC: A1.28 (ADC_6)
- net LED_G is gone; now on net TOG_2_B: A1.35 (SAI2_SCK)
- net +3V3: now also C7.1, C8.1, U4.16 (VDD), U5.16 (VDD)
- net +3V3_A: now also R5.1, U2.8 (V+)
- net +5V_USB: now also C2.1, L1.1
- net CV_1_ADC: now also A1.27 (ADC_5), U2.7; no longer A1.25 (ADC_3)
- net CV_2_ADC: now also U2.1; no longer A1.24 (ADC_2)
- net DAC_CV_1: now also U6.5 (+)
- net DAC_CV_2: now also U6.3 (+)
- net DSY_VIN: now also C49.1, R9.2
- net GND: now also C12.2, C2.2, C46.2, C49.2, C7.2, C8.2, C9.2, R32.2, R7.2, R81.1, R82.1, U2.4 (V-), U4.11 (DS), U4.8 (VSS), U5.8 (VSS), U6.4 (V-)
- net GPIO_GATEIN_1: now also A1.1 (USB_ID); no longer A1.11 (SPI1_PICO)
- net TAC_SW1: now also U5.1 (D7); no longer A1.1 (USB_ID)
- net TAC_SW2: now also U5.15 (D6); no longer A1.27 (ADC_5)
- net TOG_1: no longer A1.13 (I2C1_SDA)
- net TOG_2_B: no longer A1.8 (SPI1_CS)
- net at J_AUDIO_IN_L1.TIP, R61.2: no longer J_AUDIO_IN_R1.NORM
- net at C15.2, R37.1, R38.2: now also U2.2 (-)
- net at R49.1, R55.2: now also U6.7
- net at R48.1, R49.2: now also U6.6 (-)
- net at C14.2, R33.1, R34.2: now also U2.6 (-)
- net at R57.1, R60.2: now also U6.1
- net at R56.1, R57.2: now also U6.2 (-)
- net +12V renamed +5V_FILT
- net +5V_FILT: now also C46.1, L1.2, R8.2, R9.1, U6.8 (V+)
- net CV_3_ADC renamed SR_DIN
- net LED_B renamed SPI_SCK
- net LED_MONO_1 renamed I2C_SCL
- net LED_R renamed SPI_MOSI
- new net: C10.1, R81.2, R84.2
- new net: C10.2, R77.2
- new net: C12.1, R84.1, U1.3 (+)
- new net: R7.1, R8.1, U2.3 (+)
- new net: C11.1, R82.2, R83.1, U1.2 (-)
- new net: C11.2, R83.2, U1.1
- new net: R76.1, U2.5 (+)
- new net: C9.1, R32.1, R5.2, U1.5 (+)
- new net: U4.3 (Q7), U5.11 (DS)
- new net AREF_1V6: R76.2, U1.6 (-), U1.7
- new net AREF_2V5: R77.1
- new net I2C_SDA: A1.13 (I2C1_SDA)
- new net SPI_MISO: A1.11 (SPI1_PICO)
- new net SPI_NS: A1.8 (SPI1_CS)
- new net SR_CLK: A1.25 (ADC_3), U4.10 (CP), U5.10 (CP)
- new net SR_DATA: U5.3 (Q7)
- new net SR_LATCH: A1.24 (ADC_2), U4.9 (PL), U5.9 (PL)
- new net TAC_SW10: U4.15 (D6)
- new net TAC_SW11: U4.14 (D5)
- new net TAC_SW12: U4.13 (D4)
- new net TAC_SW13: U4.4 (D3)
- new net TAC_SW14: U4.5 (D2)
- new net TAC_SW15: U4.6 (D1)
- new net TAC_SW16: U4.7 (D0)
- new net TAC_SW3: U5.14 (D5)
- new net TAC_SW4: U5.13 (D4)
- new net TAC_SW5: U5.4 (D3)
- new net TAC_SW6: U5.5 (D2)
- new net TAC_SW7: U5.6 (D1)
- new net TAC_SW8: U5.7 (D0)
- new net TAC_SW9: U4.1 (D7)
- no-connect marks 16 -> 14
Other:
- note added: "Bias voltage for ADC Inputs"
- note added: "CV I/O"
- note added: "For this board we may want to use the inductor if it helps avoid excess voltage drop.. It'd be nice to have the addt'l filter stage prior to the seed in addition to one that cleans up the USB a bit to make +5V_FILT"
- note added: "This op-amp can be powered off 3v3A or 5V_Filt. It still has an open channel in case we need it for anything?"
- note added: "This should all move to its own "audio" page probably. Also, the OPA1652 isn't in kicad.. so I'll find one to add later"
- note added: "This version of the circuit is similar to the Field However, I am concerned about the noise from 5V USB making the ADC readings bad. See above circuit for an attempt that doesn't use the USB power directly"
- note added: "To Header (w/ 3v3 + GND)"
- note added: "Unlike buttons connected directly to the Seed, buttons connected via Shift register will need pull up resistors to 3v3 for each button. These can be found next to each button on the Peripherals Page."
- note removed: "Analog Inputs"
- moved on the sheet: A1, C17, C20, C21, C22, C3, C4, C5, J_AUDIO_IN_L1, J_AUDIO_IN_R1, J_AUDIO_OUT_L1, J_AUDIO_OUT_R1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

Commit message: sch complete (pending value changes to audio out circuit and ERC fixes), footprints set, ready for layout.
Parts:
- removed C10, C3, C5: 100NF, Capacitor_SMD:C_0603_1608Metric, symbol Device:C
- removed C11: 2.2NF, Capacitor_SMD:C_0603_1608Metric, symbol Device:C
- removed C12: 100PF, Capacitor_SMD:C_0603_1608Metric, symbol Device:C
- removed C17, C4: 330PF, Capacitor_SMD:C_0603_1608Metric, symbol Device:C
- removed C21, C22: 33PF, Capacitor_SMD:C_0603_1608Metric, symbol Device:C
- removed C9: 100UF, Capacitor_SMD:CP_Elec_6.3x7.7, symbol Device:C_Polarized_US
- removed J_AUDIO_IN_L1, J_AUDIO_IN_R1, J_AUDIO_OUT_L1, J_AUDIO_OUT_R1: ~, Electrosmith-Interface:S_JACK, symbol Electrosmith-Interface:EURO_JACK
- removed R32: 10K, Resistor_SMD:R_0603_1608Metric, symbol Seed3-Pedal-DevKit-Converted-eagle-import:Electrosmith-Passives_R-US_R0603
- removed R61, R64: 100K, Resistor_SMD:R_0603_1608Metric, symbol Device:R_US
- removed R62, R65, R67, R68, R73, R77: 10K, Resistor_SMD:R_0603_1608Metric, symbol Device:R_US
- removed R63, R66, R79, R80, R84: 100R, Resistor_SMD:R_0603_1608Metric, symbol Device:R_US
- removed R78: 100k, Resistor_SMD:R_0603_1608Metric, symbol Device:R_US
- removed R81, R83: 47K, Resistor_SMD:R_0603_1608Metric, symbol Device:R_US
- removed R82: 150R, Resistor_SMD:R_0603_1608Metric, symbol Device:R_US
- removed U1: MCP6002-xSN, symbol Amplifier_Operational:MCP6002-xSN
- added C16: 100UF, Capacitor_SMD:CP_Elec_6.3x7.7, symbol Device:C_Polarized_US
- added C18: 10UF, Capacitor_SMD:C_0805_2012Metric, symbol Device:C
- added C23, C31: 100NF, Capacitor_SMD:C_0603_1608Metric, symbol Device:C
- added R86, R87, R88: 10K, Resistor_SMD:R_0603_1608Metric, symbol Seed3-Pedal-DevKit-Converted-eagle-import:Electrosmith-Passives_R-US_R0603
- added unit 3 of U2
- added unit 2 of U6
- added unit 3 of U6
- added U9: MCP6002-xSN, Package_SO:SOIC-8_3.9x4.9mm_P1.27mm, symbol Amplifier_Operational:MCP6002-xSN
- L1: footprint (none) -> shnsly:L_SDR0805
- R5: value 10K -> 33K
- U2, U6: footprint (none) -> Package_SO:SOIC-8_3.9x4.9mm_P1.27mm
- U4, U5: footprint (none) -> Package_SO:SOIC-16_3.9x9.9mm_P1.27mm
Connections:
- net AREF_1V6 is gone; now on net +5V_FILT: R76.2
- net SR_DIN is gone; now on net SR_DATA: A1.23 (ADC_1)
- net +3V3_A: now also U2.8 (V+); no longer R5.1, U2.8 (V+)
- net +5V_FILT: now also C31.1, R88.2, U6.8 (V+), U9.8 (V+); no longer U6.8 (V+)
- net AREF_2V5: now also R86.1, U9.1, U9.2 (-)
- net DAC_CV_1: now also U6.5 (+); no longer U6.5 (+)
- net GND: now also R5.2, C16.2, C18.2, C23.2, C31.2, R86.2, R87.1, U2.4 (V-), U6.4 (V-), U9.4 (V-); no longer U2.4 (V-), U6.4 (V-)
- net at R49.1, R55.2: now also U6.7; no longer U6.7
- net at R48.1, R49.2: now also U6.6 (-); no longer U6.6 (-)
- net at R76.1, U2.5 (+): now also R5.1
- net SPI_MISO renamed SDMMC_DETECT
- net SPI_MOSI renamed AUDIO_IN_RIGHT_DETECT
- net SPI_NS: no longer names the net of A1.8 (SPI1_CS)
- net SPI_SCK renamed AUDIO_IN_LEFT_DETECT
- new net: C16.1, C18.1, C23.1, R87.2, R88.1, U9.3 (+)
- new net: U9.6 (-), U9.7
- no-connect marks 14 -> 17
Other:
- note added: "TODO: Decide if we wanna float this or GND it like usual.."
- note added: "lots of filtering for AREF_2v5"
- note removed: "AUDIO I/O"
- note removed: "Bias voltage for ADC Inputs"
- note removed: "This op-amp can be powered off 3v3A or 5V_Filt. It still has an open channel in case we need it for anything?"
- note removed: "This should all move to its own "audio" page probably. Also, the OPA1652 isn't in kicad.. so I'll find one to add later"
- note removed: "This version of the circuit is similar to the Field However, I am concerned about the noise from 5V USB making the ADC readings bad. See above circuit for an attempt that doesn't use the USB power directly"
- note removed: "To Header (w/ 3v3 + GND)"
- moved on the sheet: C14, C15, C19, C20, J_CV_IN_2, J_CV_OUT_1, J_CV_OUT_2, R33, R34, R37, R38, R48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

Commit message: lsno ERC errors or warnings, the few leftover warnings are excluded with valid comments.
Parts:
- added unit 3 of U9
- added unit 2 of U9
Connections:
- net +5V_FILT: now also U9.8 (V+); no longer U9.8 (V+)
- net GND: now also U9.4 (V-); no longer U9.4 (V-)
- new net: U9.6 (-), U9.7
Other:
- note added: "Not 100% sure why the PWR_FLAG is required here..."

Commit message: we've got a layout going
Parts:
- H1, H2, H3, H4: footprint shnsly:MNT_SLOT_M3_PLATED -> MountingHole:MountingHole_3.5mm_Pad
Changed lines of the file:
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@@
 			)
 		)
-		(property "Footprint" "shnsly:MNT_SLOT_M3_PLATED"
+		(property "Footprint" "MountingHole:MountingHole_3.5mm_Pad"
 			(at 372.11 121.92 0)
 			(effects
@@
 			)
 		)
-		(property "Footprint" "shnsly:MNT_SLOT_M3_PLATED"
+		(property "Footprint" "MountingHole:MountingHole_3.5mm_Pad"
 			(at 372.11 129.54 0)
 			(effects
@@
 			)
 		)
-		(property "Footprint" "shnsly:MNT_SLOT_M3_PLATED"
+		(property "Footprint" "MountingHole:MountingHole_3.5mm_Pad"
 			(at 372.11 137.16 0)
 			(effects
@@
 			)
 		)
-		(property "Footprint" "shnsly:MNT_SLOT_M3_PLATED"
+		(property "Footprint" "MountingHole:MountingHole_3.5mm_Pad"
 			(at 372.11 114.3 0)
 			(effects

Commit message: everything on the board -- some fine tuning necessary, and then ready to route.
Connections:
- net DAC_CV_1: now also U6.3 (+); no longer U6.5 (+)
- net DAC_CV_2: now also U6.5 (+); no longer U6.3 (+)
- net at R49.1, R55.2: now also U6.1; no longer U6.7
- net at R48.1, R49.2: now also U6.2 (-); no longer U6.6 (-)
- net at R57.1, R60.2: now also U6.7; no longer U6.1
- net at R56.1, R57.2: now also U6.6 (-); no longer U6.2 (-)
Changed lines of the file:
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@@
 		(lib_id "Amplifier_Operational:MCP6002-xSN")
 		(at 177.8 168.91 0)
-		(unit 1)
+		(unit 2)
 		(exclude_from_sim no)
 		(in_bom yes)
@@
 				(path "/19edde5c-efb5-4a72-a9f3-fb5a3c99bba0/b2297a72-db37-46bb-8b2e-2b8f47454008"
 					(reference "U6")
-					(unit 1)
+					(unit 2)
 				)
 			)
@@
 		(lib_id "Amplifier_Operational:MCP6002-xSN")
 		(at 177.8 135.89 0)
-		(unit 2)
+		(unit 1)
 		(exclude_from_sim no)
 		(in_bom yes)
@@
 				(path "/19edde5c-efb5-4a72-a9f3-fb5a3c99bba0/b2297a72-db37-46bb-8b2e-2b8f47454008"
 					(reference "U6")
-					(unit 2)
+					(unit 1)
 				)
 			)

Commit message: routed, productions mats, etc.
Parts:
- C18: value 10UF -> 10UF MLCC
Connections:
- net AUDIO_IN_LEFT_DETECT: now also A1.23 (ADC_1); no longer A1.9 (SPI1_SCK)
- net AUDIO_IN_RIGHT_DETECT: now also A1.24 (ADC_2); no longer A1.10 (SPI1_POCI)
- net SDMMC_DETECT: now also A1.8 (SPI1_CS); no longer A1.11 (SPI1_PICO)
- net SR_CLK: now also A1.9 (SPI1_SCK); no longer A1.25 (ADC_3)
- net SR_DATA: now also A1.11 (SPI1_PICO); no longer A1.23 (ADC_1)
- net SR_LATCH: now also A1.10 (SPI1_POCI); no longer A1.24 (ADC_2)
- net TOG_2_A: now also A1.35 (SAI2_SCK); no longer A1.34 (SAI2_FS)
- net TOG_2_B: now also A1.34 (SAI2_FS); no longer A1.35 (SAI2_SCK)
- new net GPIO_GATEIN_2: A1.25 (ADC_3)
- no-connect marks 17 -> 16
Changed lines of the file:
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@@
 	)
 	(no_connect
-		(at 87.63 109.22)
-	)
-	(no_connect
 		(at 266.7 175.26)
 	)
@@
 	(wire
 		(pts
+			(xy 87.63 109.22) (xy 102.87 109.22)
+		)
+		(stroke
+			(width 0)
+			(type default)
+		)
+	)
+	(wire
+		(pts
 			(xy 59.69 27.94) (xy 59.69 30.48)
 		)
@@
 	(wire
 		(pts
-			(xy 201.93 135.89) (xy 212.09 135.89)
+			(xy 31.75 106.68) (xy 36.83 106.68)
 		)
 		(stroke
@@
 	(wire
 		(pts
-			(xy 382.27 35.56) (xy 382.27 38.1)
+			(xy 201.93 135.89) (xy 212.09 135.89)
 		)
 		(stroke
@@
 	(wire
 		(pts
-			(xy 69.85 64.77) (xy 69.85 67.31)
+			(xy 382.27 35.56) (xy 382.27 38.1)
 		)
 		(stroke
@@
 	(wire
 		(pts
-			(xy 389.89 252.73) (xy 394.97 252.73)
+			(xy 69.85 64.77) (xy 69.85 67.31)
 		)
 		(stroke
@@
 	(wire
 		(pts
-			(xy 87.63 116.84) (xy 93.98 116.84)
+			(xy 389.89 252.73) (xy 394.97 252.73)
 		)
 		(stroke
@@
 	(wire
 		(pts
-			(xy 187.96 135.89) (xy 191.77 135.89)
+			(xy 87.63 116.84) (xy 93.98 116.84)
 		)
 		(stroke
@@
 	(wire
 		(pts
-			(xy 316.23 16.51) (xy 316.23 24.13)
+			(xy 187.96 135.89) (xy 191.77 135.89)
 		)
 		(stroke
@@
 	(wire
 		(pts
-			(xy 31.75 106.68) (xy 36.83 106.68)
+			(xy 316.23 16.51) (xy 316.23 24.13)
 		)
 		(stroke
@@
 	)
 	(label "SR_LATCH"
-		(at 31.75 104.14 180)
+		(at 93.98 114.3 0)
 		(effects
 			(font
 				(size 1.27 1.27)
 			)
-			(justify right bottom)
+			(justify left bottom)
 		)
 	)
@@
 		)
 	)
-	(label "SR_CLK"
-		(at 31.75 106.68 180)
-		(effects
-			(font
-				(size 1.27 1.27)
-			)
-			(justify right bottom)
-		)
-	)
 	(label "MUX_CTRL_A"
 		(at 31.75 124.46 180)
@@
 		)
 	)
+	(label "SR_CLK"
+		(at 93.98 111.76 0)
+		(effects
+			(font
+				(size 1.27 1.27)
+			)
+			(justify left bottom)
+		)
+	)
 	(label "SR_DATA"
-		(at 31.75 101.6 180)
+		(at 93.98 116.84 0)
 		(effects
 			(font
 				(size 1.27 1.27)
 			)
-			(justify right bottom)
+			(justify left bottom)
 		)
 	)
@@
 	(global_label "AUDIO_IN_LEFT_DETECT"
 		(shape input)
-		(at 93.98 111.76 0)
+		(at 31.75 101.6 180)
 		(fields_autoplaced yes)
 		(effects
@@
 				(size 1.27 1.27)
 			)
-			(justify left)
+			(justify right)
 		)
 		(property "Intersheetrefs" "${INTERSHEET_REFS}"
-			(at 118.4342 111.76 0)
+			(at 7.2958 101.6 0)
 			(effects
 				(font
 					(size 1.27 1.27)
 				)
-				(justify left)
+				(justify right)
 				(hide yes)
 			)
@@
 	(global_label "SDMMC_DETECT"
 		(shape input)
-		(at 93.98 116.84 0)
+		(at 102.87 109.22 0)
 		(fields_autoplaced yes)
 		(effects
@@
 		)
 		(property "Intersheetrefs" "${INTERSHEET_REFS}"
-			(at 111.3583 116.84 0)
+			(at 120.2483 109.22 0)
 			(effects
 				(font
@@
 		)
 	)
+	(global_label "GPIO_GATEIN_2"
+		(shape bidirectional)
+		(at 31.75 106.68 180)
+		(fields_autoplaced yes)
+		(effects
+			(font
+				(size 1.2446 1.2446)
+			)
+			(justify right)
+		)
+		(property "Intersheetrefs" "${INTERSHEET_REFS}"
+			(at 13.9857 106.68 0)
+			(effects
+				(font
+					(size 1.27 1.27)
+				)
+				(justify right)
+				(hide yes)
+			)
+		)
+	)
 	(global_label "MIDI_RX"
 		(shape input)
@@
 	(global_label "TOG_2_B"
 		(shape bidirectional)
-		(at 31.75 134.62 180)
+		(at 31.75 132.08 180)
 		(fields_autoplaced yes)
 		(effects
@@
 		)
 		(property "Intersheetrefs" "${INTERSHEET_REFS}"
-			(at 19.9125 134.62 0)
+			(at 20.0903 132.08 0)
 			(effects
 				(font
@@
 	(global_label "AUDIO_IN_RIGHT_DETECT"
 		(shape input)
-		(at 93.98 114.3 0)
+		(at 31.75 104.14 180)
 		(fields_autoplaced yes)
 		(effects
@@
 				(size 1.27 1.27)
 			)
-			(justify left)
+			(justify right)
 		)
 		(property "Intersheetrefs" "${INTERSHEET_REFS}"
-			(at 119.6438 114.3 0)
+			(at 6.0862 104.14 0)
 			(effects
 				(font
 					(size 1.27 1.27)
 				)
-				(justify left)
+				(justify right)
 				(hide yes)
 			)
@@
 	(global_label "TOG_2_A"
 		(shape bidirectional)
-		(at 31.75 132.08 180)
+		(at 31.75 134.62 180)
 		(fields_autoplaced yes)
 		(effects
@@
 		)
 		(property "Intersheetrefs" "${INTERSHEET_REFS}"
-			(at 20.0903 132.08 0)
+			(at 19.9125 134.62 0)
 			(effects
 				(font
@@
 		(dnp no)
 		(property "Reference" "C18"
-			(at 107.95 21.5899 0)
+			(at 110.49 27.432 0)
 			(effects
 				(font
@@
 			)
 		)
-		(property "Value" "10UF"
-			(at 107.95 24.1299 0)
+		(property "Value" "10UF MLCC"
+			(at 107.95 25.908 90)
 			(effects
 				(font
