File: pcb/ES-Seed3-DevKit-Desktop-Rev2/audio.kicad_sch (KiCad schematic)
At the start: 49 parts, among them J1 AudioJack3_Switch, J2 AudioJack3_Switch, J3 AudioJack3_Switch, J4 AudioJack3_Switch, J5 AudioJack3_Switch_HEADPHONE, U1 TPA6110A2DGN, U15 OPA1652, U3 OPA1652

Commit message: layout and routing for changes -- need to review, and make mats.
Connections:
- net +5V_FILT: no longer C3.2, C5.2, U15.8 (V+), U3.8 (V+)
- net AREF_2V5 renamed AREF_AUDIO_BIAS
- new net +9V_A: C3.2, C5.2, U15.8 (V+), U3.8 (V+)
Other:
- note added: "DECISION - Two Choices: 1. Add LD1117 (or LP2985) or other 5V Linear Reg. 2. Power TPA6110 from Seed's 3v3A"
- note added: "Detection nets should _probably_ get a pair of diodes for protection.."
- moved on the sheet: C26, C4, R61, R96

Commit message: a few more changes, and regenerated production mats
Parts:
- added C42, C43: 10UF, Capacitor_SMD:CP_Elec_4x5.8, symbol Device:C_Polarized
- added R100, R101: 10K, Resistor_SMD:R_0603_1608Metric, symbol Device:R_US
- added R102, R103: 100R, Resistor_SMD:R_0603_1608Metric, symbol Device:R_US
- C13, C25: value 330PF -> 330PF C0G
- C17, C27: value 470PF -> 470PF C0G
Connections:
- net CODEC_OUT_L: now also C42.2; no longer R61.2
- net CODEC_OUT_R: now also C43.2; no longer R96.2
- net GND: now also R100.2, R101.2
- net at C17.1, R63.1, U3.7: now also R102.1; no longer C12.1
- net at C27.1, R94.1, U3.1: now also R103.1; no longer C11.1
- net at C12.2, J3.T: now also R101.1
- net at C11.2, J4.T: now also R100.1
- new net: C11.1, R103.2
- new net: C12.1, R102.2
- new net: C42.1, R61.2
- new net: C43.1, R96.2
Other:
- moved on the sheet: C11, C12, J3, J4
