File: pcb/ES-Seed3-DevKit-Desktop-Rev2/ES-Seed3-DevKit-Desktop-Rev2.kicad_pcb (KiCad board)
At the start: 2 copper layers, 197 x 111 mm, 214 parts, among them J1 AudioJack3_Switch, J10 DIN_MIDI_5P, J11 DIN_MIDI_5P, J2 AudioJack3_Switch, J3 AudioJack3_Switch, J4 AudioJack3_Switch, J5 AudioJack3_Switch_HEADPHONE, J7 USB4110GFA, J8 DIN_MIDI_5P, Q1 MMBT3904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

Commit message: layout and routing for changes -- need to review, and make mats.
Parts:
- removed L1: 1mH, shnsly:L_SDR0805
- added C33: 10UF MLCC, Capacitor_SMD:C_0805_2012Metric, F.Cu at (59.6, 74.1)
- added C35: 10UF MLCC, Capacitor_SMD:C_0805_2012Metric, F.Cu at (59.7, 64.9)
- added C36: 560PF, Capacitor_SMD:C_0603_1608Metric, F.Cu at (53.3, 66.6)
- added C37: 100UF, Capacitor_SMD:CP_Elec_6.3x7.7, F.Cu at (73.0, 64.5)
- added C38: 100UF, Capacitor_SMD:CP_Elec_6.3x7.7, F.Cu at (73.0, 72.5)
- added C39: 100UF, Capacitor_SMD:CP_Elec_6.3x7.7, F.Cu at (73.0, 80.5)
- added C40: 100NF, Capacitor_SMD:C_0603_1608Metric, F.Cu at (73.0, 87.2)
- added C41: 100UF, Capacitor_SMD:CP_Elec_6.3x7.7, F.Cu at (90.5, 80.5)
- added D17: 1N5817WS, Diode_SMD:D_SOD-323F, F.Cu at (56.8, 66.5)
- added D18: 1N5817WS, Diode_SMD:D_SOD-323F, F.Cu at (98.5, 106.5)
- added D19: 1N5817WS, Diode_SMD:D_SOD-323F, F.Cu at (94.5, 106.5)
- added D20: 1N5817WS, Diode_SMD:D_SOD-323F, F.Cu at (125.5, 59.0)
- added D25: 1N5817WS, Diode_SMD:D_SOD-323F, F.Cu at (125.5, 64.5)
- added L2: 6.8uH 2.9A, Inductor_SMD:L_TDK_VLS6045EX_VLS6045AF, F.Cu at (61.2, 69.4)
- added R81: 1M, Resistor_SMD:R_0603_1608Metric, F.Cu at (56.0, 73.4)
- added R82: 62K, Resistor_SMD:R_0603_1608Metric, F.Cu at (54.9, 66.6)
- added R83: 10K, Resistor_SMD:R_0603_1608Metric, F.Cu at (53.3, 69.9)
- added R84: 0R, Resistor_SMD:R_0603_1608Metric, F.Cu at (56.0, 75.0)
- added R95: 3R3, Resistor_SMD:R_1206_3216Metric, F.Cu at (62.6, 94.8)
- added R97: 3R3, Resistor_SMD:R_1206_3216Metric, F.Cu at (67.5, 68.5)
- added R98: 3R3, Resistor_SMD:R_1206_3216Metric, F.Cu at (67.5, 76.5)
- added R99: 3R3, Resistor_SMD:R_1206_3216Metric, F.Cu at (86.5, 86.0)
- added U10: LD1117S50TR_SOT223, Package_TO_SOT_SMD:SOT-223-3_TabPin2, F.Cu at (77.5, 89.8)
- added U7: LMR62421XMF, Package_TO_SOT_SMD:SOT-23-5, F.Cu at (56.0, 70.5)
- moved LOGO1 107.0 mm to (167.2, 87.4)
- moved C2 12.3 mm to (82.5, 80.5)
- moved R86 11.5 mm to (76.5, 96.5), turned to 180 degrees
- moved U9 10.3 mm to (82.0, 97.5), turned to 0 degrees
- moved R87 9.06 mm to (69.0, 90.0), turned to -90 degrees
- moved C16 8.74 mm to (70.5, 99.0), turned to 180 degrees
- moved C31 7.87 mm to (84.0, 94.0), turned to 180 degrees
- moved R88 7.38 mm to (70.6, 90.0), turned to 90 degrees
- moved C23 6.46 mm to (69.8, 92.4), turned to 180 degrees
- moved C18 6.38 mm to (69.6, 94.2), turned to 180 degrees
Connections:
- net AREF_2V5 renamed AREF_AUDIO_BIAS
- C2 pad 1: /Daisy/+5V_USB -> Net-(U10-VO)
- C3 pad 2: +5V_FILT -> +9V_A
- C46 pad 1: +5V_FILT -> Net-(C46-Pad1)
- C5 pad 2: +5V_FILT -> +9V_A
- R88 pad 2: +5V_FILT -> +9V_A
- R9 pad 1: +5V_FILT -> Net-(C46-Pad1)
- U12 pad 6: unconnected-(U12-INH-Pad6) -> GND
- U15 pad 8: +5V_FILT -> +9V_A
- U3 pad 8: +5V_FILT -> +9V_A
- U8 pad 23: +3V3 -> GND
Routing:
- net +9V_A: track 0.00 -> 200.3 mm, vias 0 -> 4
- net BOOST_VCC: track 0.00 -> 59.9 mm
- net +5V_FILT: track 290.6 -> 245.9 mm, vias 8 -> 7
- net +3V3: track 526.1 -> 559.1 mm
- net Net-(U10-VO): track 0.00 -> 18.2 mm
- net AREF_AUDIO_BIAS: track 145.9 -> 156.7 mm
- net Net-(U7-VIN): track 0.00 -> 9.60 mm
- net Net-(C38-Pad1): track 0.00 -> 9.40 mm
- net Net-(C46-Pad1): track 0.00 -> 8.93 mm
- net Net-(D17-A): track 0.00 -> 6.35 mm
- net AUDIO_IN_LEFT_DETECT: track 177.0 -> 182.7 mm
- net Net-(U7-FB): track 0.00 -> 5.19 mm
- net AUDIO_IN_RIGHT_DETECT: track 156.4 -> 161.5 mm
- net Net-(J_CV_OUT_1-PadTIP): track 25.5 -> 22.5 mm
- net /Daisy/+5V_USB: track 29.4 -> 32.3 mm
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
Commit message: a few more changes, and regenerated production mats
Parts:
- added C42: 10UF, Capacitor_SMD:CP_Elec_4x5.8, F.Cu at (118.8, 80.8)
- added C43: 10UF, Capacitor_SMD:CP_Elec_4x5.8, F.Cu at (98.9, 86.1)
- added QR1: ~, shnsly:qr-seed3-desktop-redirect-medium, F.Cu at (66.4, 50.7)
- added R100: 10K, Resistor_SMD:R_0603_1608Metric, F.Cu at (97.5, 75.8)
- added R101: 10K, Resistor_SMD:R_0603_1608Metric, F.Cu at (115.6, 75.8)
- added R102: 100R, Resistor_SMD:R_0603_1608Metric, F.Cu at (111.4, 80.4)
- added R103: 100R, Resistor_SMD:R_0603_1608Metric, F.Cu at (100.6, 79.2)
- C13, C25: value 330PF -> 330PF C0G
- C17, C27: value 470PF -> 470PF C0G
- moved C12 1.39 mm to (110.5, 75.8), turned to 0 degrees
- moved C11 1.31 mm to (102.4, 75.8), turned to 180 degrees
Connections:
- C17 pad 1: Net-(C12-Pad1) -> Net-(C17-Pad1)
- C27 pad 1: Net-(C11-Pad1) -> Net-(C27-Pad1)
- R61 pad 2: CODEC_OUT_L -> Net-(C42-Pad1)
- R63 pad 1: Net-(C12-Pad1) -> Net-(C17-Pad1)
- R94 pad 1: Net-(C11-Pad1) -> Net-(C27-Pad1)
- R96 pad 2: CODEC_OUT_R -> Net-(C43-Pad1)
- U3 pad 1: Net-(C11-Pad1) -> Net-(C27-Pad1)
- U3 pad 7: Net-(C12-Pad1) -> Net-(C17-Pad1)
Routing:
- net Net-(C42-Pad1): track 0.00 -> 6.52 mm
- net Net-(C43-Pad1): track 0.00 -> 6.31 mm
- net Net-(C17-Pad1): track 0.00 -> 5.44 mm
- net Net-(C27-Pad1): track 0.00 -> 5.37 mm
- net Net-(C12-Pad2): track 13.6 -> 17.3 mm
- net CODEC_OUT_L: track 238.8 -> 242.0 mm
- net CODEC_OUT_R: track 219.1 -> 216.9 mm
- net Net-(C11-Pad1): track 6.20 -> 4.61 mm
- net Net-(C12-Pad1): track 7.63 -> 6.13 mm
- net CODEC_IN_L: track 163.9 -> 162.5 mm
- net /Daisy/POT_MUX: track 54.3 -> 53.2 mm
- net CODEC_IN_R: track 152.4 -> 153.0 mm
- net GND: vias 26 -> 35
Other:
- board text added: "Rev2"
- board text removed: "Rev1"

Commit message: updated values for CD4021, and regenerated mats.
Parts:
- U4, U5: value 4021 -> CD4021BM96
Changed lines of the file:
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@@
 			)
 		)
-		(property "Value" "4021"
+		(property "Value" "CD4021BM96"
 			(at 0 5.9 0)
 			(layer "F.Fab")
@@
 			)
 		)
-		(property "Value" "4021"
+		(property "Value" "CD4021BM96"
 			(at 0 5.9 0)
 			(layer "F.Fab")
