File: pcb/ES-Seed3-DevKit-Desktop-Rev3/ES-Seed3-DevKit-Desktop-Rev3.kicad_pcb (KiCad board)
At the start: 2 copper layers, 197 x 111 mm, 238 parts, among them J1 AudioJack3_Switch, J10 DIN_MIDI_5P, J11 DIN_MIDI_5P, J2 AudioJack3_Switch, J3 AudioJack3_Switch, J4 AudioJack3_Switch, J5 AudioJack3_Switch_HEADPHONE, J7 USB4110GFA, J8 DIN_MIDI_5P, Q1 MMBT3904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

Commit message: added board characteristics, and regen'd prod
Routing:
- net Net-(J7-CC2): track 4.13 -> 5.98 mm

Commit message: updated rev text.
Other:
- board text added: "Rev3"
- board text removed: "Rev2"
Changed lines of the file:
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@@
 		)
 	)
-	(gr_text "Rev2"
+	(gr_text "Rev3"
 		(at 74 47.6 0)
 		(layer "B.SilkS")
