File: pcb/ES-Seed3-DevKit-Desktop-Rev3/audio.kicad_sch (KiCad schematic)
At the start: 55 parts, among them J1 AudioJack3_Switch, J2 AudioJack3_Switch, J3 AudioJack3_Switch, J4 AudioJack3_Switch, J5 AudioJack3_Switch_HEADPHONE, U1 TPA6110A2DGN, U15 OPA1652, U3 OPA1652

Commit message: schematic level changes for fixing CV idle offset, and audio whine tone.
Parts:
- removed D21, D22, D23, D24: 1N5817WS, Diode_SMD:D_SOD-323F, symbol Device:D_Schottky
- removed R64, R65: 47K, Resistor_SMD:R_0603_1608Metric, symbol Device:R_US

Commit message: partial directory update for cleanup of schematic comments after validating rev3 HW
Other:
- note removed: "DECISION - Two Choices: 1. Add LD1117 (or LP2985) or other 5V Linear Reg. 2. Power TPA6110 from Seed's 3v3A"
- note removed: "Detection nets should _probably_ get a pair of diodes for protection.."
- note removed: "Gain is set to target +4dBu (maximum) obviously this does not make it a pro-line-level device that way.. we'd need to probably have a certain amount of headroom. If, instead we look at this as a -10dBV device, then we have ~14dB of headroom with these values. Gin=0.814 (Rin=10k, Rfb=16k) Gout=1.228 (Rin=10k, Rfb=24k) Alternatively we can go closer to the PCM3060's "2Vrms" reference and just do: G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"
- note removed: "I updated these to be gain of 2. However, I'm not really sure how the math works out for the other two values.. So, I may just need to kludge those a a bit IRL. (This can also be reworked to be our normal basic filter)"
Changed lines of the file:
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@@
 	(generator_version "9.0")
 	(paper "A4")
-	(text "Gain is set to target +4dBu (maximum)\nobviously this does not make it a pro-line-level device that way..\nwe'd need to probably have a certain amount of headroom.\nIf, instead we look at this as a -10dBV device, then we have\n~14dB of headroom with these values.\n\nGin=0.814 (Rin=10k, Rfb=16k)\nGout=1.228 (Rin=10k, Rfb=24k)\n\nAlternatively we can go closer to the PCM3060's \"2Vrms\" reference and just do:\nGin=0.5, Gout=2 :shrug:\n\nFor now, I've implemented the left channel of audio with less atten/gain."
-		(exclude_from_sim no)
-		(at 5.08 170.942 0)
-		(effects
-			(font
-				(size 1.27 1.27)
-			)
-			(justify left)
-		)
-	)
-	(text "I updated these to be gain of 2.\nHowever, I'm not really sure how the math works out for the other two values..\nSo, I may just need to kludge those a a bit IRL.\n(This can also be reworked to be our normal basic filter)"
-		(exclude_from_sim no)
-		(at 256.794 62.484 0)
-		(effects
-			(font
-				(size 1.27 1.27)
-			)
-		)
-	)
-	(text "Detection nets should _probably_ get a pair of diodes for protection.."
-		(exclude_from_sim no)
-		(at 21.59 52.578 0)
-		(effects
-			(font
-				(size 1.27 1.27)
-			)
-		)
-	)
 	(text "AUDIO I/O"
 		(exclude_from_sim no)
@@
 			)
 		)
-	)
-	(text "DECISION - Two Choices:\n1. Add LD1117 (or LP2985) or other 5V Linear Reg.\n2. Power TPA6110 from Seed's 3v3A"
-		(exclude_from_sim no)
-		(at 244.602 127.762 0)
-		(effects
-			(font
-				(size 1.27 1.27)
-			)
-		)
